Commit message: parse error fixed

File: lpv_description/urdf/lpv_base.urdf.xacro (robot description, xacro)
@@ -98,4 +98,5 @@
     </gazebo>
     <visual>
+      <origin xyz="0 -0 -0.6" rpy="0 0 0" />
       <geometry>
         <mesh filename="package://lpv_description/models/LPV-Base/mesh/lpv_base.dae" scale="0.05 0.05 0.05"/>

File: lpv_gazebo/urdf/components/lpv_radar.xacro (robot description, xacro)
@@ -2,5 +2,5 @@
 <robot xmlns:xacro="http://ros.org/wiki/xacro">
   <xacro:macro name="lpv_radar" params="name:=radar x:=0.6 y:=0 z:=0.95
-				       R:=0 P:=0 Y:=pi update_rate:=10">
+				       R:=0 P:=0 Y:=0 update_rate:=10">
 				       <!-- Links-->
     <link name="${namespace}/${name}_link">

File: lpv_gazebo/urdf/dynamics/lpv_gazebo_dynamics_plugin.xacro (robot description, xacro)
@@ -1,5 +1,5 @@
 <?xml version="1.0"?>
 <robot xmlns:xacro="http://ros.org/wiki/xacro">
-  <xacro:macro name="usv_dynamics_gazebo" params="name width:=1.2 length:=3">
+  <xacro:macro name="usv_dynamics_gazebo" params="name width:=2.9 length:=4.9">
     <!--Gazebo Plugin for simulating WAM-V dynamics-->
     <gazebo>

File: lpv_gazebo/urdf/lpv_gazebo.urdf.xacro (robot description, xacro)
@@ -97,5 +97,5 @@
     <!-- Add simulated GPS -->
     <xacro:if value="$(arg gps_enabled)">
-      <xacro:lpv_gps name="lpv_gps" x="-0.85" />
+      <xacro:lpv_gps name="gps_lpv" x="-0.85" />
     </xacro:if>
     <!-- Add P3D ground truth -->
@@ -110,9 +110,9 @@
     <xacro:if value="$(arg aimm_sensors_enabled)">
       <!-- Add a stereo camera pair -->
-      <xacro:lpv_camera name="front_left_camera" y="0.7" x="-3" z="1.2" P="${radians(0)}" Y="${radians(120)}" post_Y="${radians(120)}" visualize="true"/>
-      <xacro:lpv_camera name="front_right_camera" y="-0.7" x="-3" z="1.2" P="${radians(0)}" Y="${radians(-120)}" post_Y="${radians(-120)}" visualize="true"/>
+      <xacro:lpv_camera name="front_left_camera" y="0.7" x="-3" z="0.9" P="${radians(0)}" Y="${radians(120)}" post_Y="${radians(120)}" visualize="true"/>
+      <xacro:lpv_camera name="front_right_camera" y="-0.7" x="-3" z="0.9" P="${radians(0)}" Y="${radians(-120)}" post_Y="${radians(-120)}" visualize="true"/>
       <!-- Add simulated GPS + Radar -->
-      <xacro:lpv_gps name="gps_lpv" x="0"/>
-      <xacro:lpv_radar name="radar_lpv" x="-0.85" />
+      <xacro:lpv_gps name="gps_lpv" x="0.3" z="0.8"/>
+      <xacro:lpv_radar name="radar_lpv" x="-0.85" y="0" z="0.9" P="${radians(0)}" Y="${radians(-180)}"  />
     </xacro:if>
   </xacro:unless>
